Commit message: rx60_description verbessert

File: src/rx60_description/urdf/rx60.urdf.xacro (robot description, xacro)
@@ -1,4 +1,7 @@
 <?xml version="1.0"?>
-<robot name="rx60" xmlns:xacro="http://www.ros.org/wiki/xacro">
+<robot name="rx60" xmlns:xacro="http://ros.org/wiki/xacro">
+  <!-- Import transmission and gazebo elements -->
+  <xacro:include filename="$(find rx60_description)/urdf/rx60.transmission.xacro"/>
+  <xacro:include filename="$(find rx60_description)/urdf/rx60.gazebo.xacro"/>
   <!-- Links -->
   <link name="base_link">
@@ -199,6 +202,6 @@
     <child link="shoulder_link"/>
     <axis xyz="0 0 1"/>
-    <limit lower="-2.7925" upper="2.7925" velocity="0.5" effort="1000"/>
-    <dynamics friction="0.0001" damping="1"/>
+    <limit lower="-2.7925" upper="2.7925" velocity="5" effort="330.0"/>
+    <dynamics friction="0.001" damping="1"/>
   </joint>
   <joint name="joint2" type="revolute">
@@ -207,6 +210,6 @@
     <child link="arm_link"/>
     <axis xyz="0 0 1"/>
-    <limit lower="-2.2253" upper="2.2253" velocity="0.5" effort="1000"/>
-    <dynamics friction="0.0001" damping="1"/>
+    <limit lower="-2.2253" upper="2.2253" velocity="5" effort="330.0"/>
+    <dynamics friction="0.001" damping="1"/>
   </joint>
   <joint name="joint3" type="revolute">
@@ -215,6 +218,6 @@
     <child link="elbow_link"/>
     <axis xyz="0 0 1"/>
-    <limit lower="-2.3474" upper="2.3474" velocity="0.5" effort="1000"/>
-    <dynamics friction="0.0001" damping="1"/>
+    <limit lower="-2.3474" upper="2.3474" velocity="5.5" effort="150.0"/>
+    <dynamics friction="0.001" damping="1"/>
   </joint>
   <joint name="joint4" type="revolute">
@@ -223,6 +226,6 @@
     <child link="forearm_link"/>
     <axis xyz="0 0 1"/>
-    <limit lower="-4.7123" upper="4.7123" velocity="0.5" effort="1000"/>
-    <dynamics friction="0.0001" damping="1"/>
+    <limit lower="-4.7123" upper="4.7123" velocity="7.1" effort="54.0"/>
+    <dynamics friction="0.001" damping="1"/>
   </joint>
   <joint name="joint5" type="revolute">
@@ -231,6 +234,6 @@
     <child link="wrist_link"/>
     <axis xyz="0 0 1"/>
-    <limit lower="-1.9111" upper="2.1031" velocity="0.5" effort="1000"/>
-    <dynamics friction="0.0001" damping="1"/>
+    <limit lower="-1.9111" upper="2.1031" velocity="5.5" effort="54.0"/>
+    <dynamics friction="0.001" damping="1"/>
   </joint>
   <joint name="joint6" type="revolute">
@@ -239,75 +242,6 @@
     <child link="tool_link"/>
     <axis xyz="0 0 1"/>
-    <limit lower="-4.7124" upper="4.7124" velocity="0.5" effort="1000"/>
-    <dynamics friction="0.0001" damping="1"/>
-  </joint>
-  <!-- Transmissions -->
-  <transmission name="joint1_trans">
-    <type>transmission_interface/SimpleTransmission</type>
-    <joint name="joint1">
-      <hardwareInterface>hardware_interface/EffortJointInterface</hardwareInterface>
-    </joint>
-    <actuator name="motor1">
-      <hardwareInterface>EffortJointInterface</hardwareInterface>
-      <mechanicalReduction>30</mechanicalReduction>  <!-- geschaetzter Wert -->
-    </actuator>
-  </transmission>
-  <transmission name="joint2_trans">
-    <type>transmission_interface/SimpleTransmission</type>
-    <joint name="joint2">
-      <hardwareInterface>hardware_interface/EffortJointInterface</hardwareInterface>
-    </joint>
-    <actuator name="motor2">
-      <hardwareInterface>EffortJointInterface</hardwareInterface>
-      <mechanicalReduction>30</mechanicalReduction>  <!-- geschaetzter Wert -->
-    </actuator>
-  </transmission>
-  <transmission name="joint3_trans">
-    <type>transmission_interface/SimpleTransmission</type>
-    <joint name="joint3">
-      <hardwareInterface>hardware_interface/EffortJointInterface</hardwareInterface>
-    </joint>
-    <actuator name="motor3">
-      <hardwareInterface>EffortJointInterface</hardwareInterface>
-      <mechanicalReduction>30</mechanicalReduction>  <!-- geschaetzter Wert -->
-    </actuator>
-  </transmission>
-  <transmission name="joint4_trans">
-    <type>transmission_interface/SimpleTransmission</type>
-    <joint name="joint4">
-      <hardwareInterface>hardware_interface/EffortJointInterface</hardwareInterface>
-    </joint>
-    <actuator name="motor4">
-      <hardwareInterface>EffortJointInterface</hardwareInterface>
-      <mechanicalReduction>15</mechanicalReduction>  <!-- geschaetzter Wert -->
-    </actuator>
-  </transmission>
-  <transmission name="joint5_trans">
-    <type>transmission_interface/SimpleTransmission</type>
-    <joint name="joint5">
-      <hardwareInterface>hardware_interface/EffortJointInterface</hardwareInterface>
-    </joint>
-    <actuator name="motor5">
-      <hardwareInterface>EffortJointInterface</hardwareInterface>
-      <mechanicalReduction>15</mechanicalReduction>  <!-- geschaetzter Wert -->
-    </actuator>
-  </transmission>
-  <transmission name="joint6_trans">
-    <type>transmission_interface/SimpleTransmission</type>
-    <joint name="joint6">
-      <hardwareInterface>hardware_interface/EffortJointInterface</hardwareInterface>
-    </joint>
-    <actuator name="motor6">
-      <hardwareInterface>EffortJointInterface</hardwareInterface>
-      <mechanicalReduction>15</mechanicalReduction>  <!-- geschaetzter Wert -->
-    </actuator>
-  </transmission>
-  <!-- base_link an Gazebo world fixieren -->
-  <link name="world"/>
-  <joint name="fixed" type="fixed">
-    <parent link="world"/>
-    <child link="base_link"/>
-  </joint>
-  <!-- Import all Gazebo-customization elements -->
-  <xacro:include filename="$(find rx60_description)/urdf/rx60.gazebo" />
+    <limit lower="-4.7124" upper="4.7124" velocity="12.2" effort="32.0"/>
+    <dynamics friction="0.001" damping="1"/>
+  </joint>
 </robot>
